File: kicad/pcb/keys.kicad_sch (KiCad schematic)
At the start: 116 parts

Commit message: USB (almost) done + some STM progress
Other:
- added sheet RGB (rgb.kicad_sch)

Commit message: (WIP) Tracing v2
Connections:
- net COL_0: now also MX1.2, MX13.2, MX25.2, MX37.2, MX49.2; no longer MX1.1, MX13.1, MX25.1, MX37.1, MX49.1
- net COL_1: now also MX14.2, MX2.2, MX26.2, MX38.2, MX50.2; no longer MX14.1, MX2.1, MX26.1, MX38.1, MX50.1
- net COL_10: now also MX11.2, MX23.2, MX35.2, MX47.2, MX57.2; no longer MX11.1, MX23.1, MX35.1, MX47.1, MX57.1
- net COL_11: now also MX12.2, MX24.2, MX36.2, MX48.2, MX58.2; no longer MX12.1, MX24.1, MX36.1, MX48.1, MX58.1
- net COL_2: now also MX15.2, MX27.2, MX3.2, MX39.2, MX51.2; no longer MX15.1, MX27.1, MX3.1, MX39.1, MX51.1
- net COL_3: now also MX16.2, MX28.2, MX4.2, MX40.2, MX52.2; no longer MX16.1, MX28.1, MX4.1, MX40.1, MX52.1
- net COL_4: now also MX17.2, MX29.2, MX41.2, MX5.2, MX53.2; no longer MX17.1, MX29.1, MX41.1, MX5.1, MX53.1
- net COL_5: now also MX18.2, MX30.2, MX42.2, MX6.2; no longer MX18.1, MX30.1, MX42.1, MX6.1
- net COL_6: now also MX19.2, MX31.2, MX43.2, MX54.2, MX7.2; no longer MX19.1, MX31.1, MX43.1, MX54.1, MX7.1
- net COL_7: now also MX20.2, MX32.2, MX44.2, MX8.2; no longer MX20.1, MX32.1, MX44.1, MX8.1
- net COL_8: now also MX21.2, MX33.2, MX45.2, MX55.2, MX9.2; no longer MX21.1, MX33.1, MX45.1, MX55.1, MX9.1
- net COL_9: now also MX10.2, MX22.2, MX34.2, MX46.2, MX56.2; no longer MX10.1, MX22.1, MX34.1, MX46.1, MX56.1
- net at D48.2 (A): now also MX48.1; no longer MX48.2
- net at D21.2 (A): now also MX21.1; no longer MX21.2
- net at D3.2 (A): now also MX3.1; no longer MX3.2
- net at D33.2 (A): now also MX33.1; no longer MX33.2
- net at D4.2 (A): now also MX4.1; no longer MX4.2
- net at D30.2 (A): now also MX30.1; no longer MX30.2
- net at D18.2 (A): now also MX18.1; no longer MX18.2
- net at D46.2 (A): now also MX46.1; no longer MX46.2
- net at D57.2 (A): now also MX57.1; no longer MX57.2
- net at D24.2 (A): now also MX24.1; no longer MX24.2
- net at D39.2 (A): now also MX39.1; no longer MX39.2
- net at D38.2 (A): now also MX38.1; no longer MX38.2
- net at D37.2 (A): now also MX37.1; no longer MX37.2
- net at D19.2 (A): now also MX19.1; no longer MX19.2
- net at D47.2 (A): now also MX47.1; no longer MX47.2
- net at D14.2 (A): now also MX14.1; no longer MX14.2
- net at D28.2 (A): now also MX28.1; no longer MX28.2
- net at D49.2 (A): now also MX49.1; no longer MX49.2
- net at D32.2 (A): now also MX32.1; no longer MX32.2
- net at D25.2 (A): now also MX25.1; no longer MX25.2
- net at D29.2 (A): now also MX29.1; no longer MX29.2
- net at D40.2 (A): now also MX40.1; no longer MX40.2
- net at D50.2 (A): now also MX50.1; no longer MX50.2
- net at D51.2 (A): now also MX51.1; no longer MX51.2
- net at D34.2 (A): now also MX34.1; no longer MX34.2
- net at D13.2 (A): now also MX13.1; no longer MX13.2
- net at D20.2 (A): now also MX20.1; no longer MX20.2
- net at D7.2 (A): now also MX7.1; no longer MX7.2
- net at D58.2 (A): now also MX58.1; no longer MX58.2
- net at D42.2 (A): now also MX42.1; no longer MX42.2
- net at D41.2 (A): now also MX41.1; no longer MX41.2
- net at D1.2 (A): now also MX1.1; no longer MX1.2
- net at D9.2 (A): now also MX9.1; no longer MX9.2
- net at D55.2 (A): now also MX55.1; no longer MX55.2
- net at D10.2 (A): now also MX10.1; no longer MX10.2
- net at D36.2 (A): now also MX36.1; no longer MX36.2
- net at D53.2 (A): now also MX53.1; no longer MX53.2
- net at D6.2 (A): now also MX6.1; no longer MX6.2
- net at D44.2 (A): now also MX44.1; no longer MX44.2
- net at D2.2 (A): now also MX2.1; no longer MX2.2
- net at D5.2 (A): now also MX5.1; no longer MX5.2
- net at D43.2 (A): now also MX43.1; no longer MX43.2
- net at D22.2 (A): now also MX22.1; no longer MX22.2
- net at D12.2 (A): now also MX12.1; no longer MX12.2
- net at D23.2 (A): now also MX23.1; no longer MX23.2
- net at D27.2 (A): now also MX27.1; no longer MX27.2
- net at D8.2 (A): now also MX8.1; no longer MX8.2
- net at D35.2 (A): now also MX35.1; no longer MX35.2
- net at D54.2 (A): now also MX54.1; no longer MX54.2
- net at D15.2 (A): now also MX15.1; no longer MX15.2
- net at D31.2 (A): now also MX31.1; no longer MX31.2
- net at D16.2 (A): now also MX16.1; no longer MX16.2
- net at D26.2 (A): now also MX26.1; no longer MX26.2
- net at D45.2 (A): now also MX45.1; no longer MX45.2
- net at D11.2 (A): now also MX11.1; no longer MX11.2
- net at D17.2 (A): now also MX17.1; no longer MX17.2
- net at D52.2 (A): now also MX52.1; no longer MX52.2
- net at D56.2 (A): now also MX56.1; no longer MX56.2
Other:
- moved on the sheet: MX1, MX10, MX11, MX12, MX13, MX14, MX15, MX16, MX17, MX18, MX19, MX2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
