File: kicad/pcb/pcb.kicad_pcb (KiCad board)
At the start: 2 copper layers, 274.7 x 100.5 mm, 235 parts, among them U1 FE1.1, U2 STM32H750VBTx, U3 ESP32-S3-WROOM-2

Commit message: USB (almost) done + some STM progress
Parts:
- added U5: MIC2026-2BM, Package_DIP:DIP-8_W7.62mm, F.Cu at (244.2, 161.4)
- added U6: USBLC6-2P6, Package_TO_SOT_SMD:SOT-666, F.Cu at (255.4, 161.0)
- C1, C10, C11, C12, C13, C14, C15, C16, C17, C18, C19, C2, C20, C21, C22, C23, C24, C25, C26, C27, C28, C29, C3, C30, C31, C32, C33, C34, C35, C36, C37, C38, C39, C4, C40, C41, C42, C43, C44, C45, C46, C47, C48, C49, C5, C50, C51, C52, C53, C54, C55, C56, C57, C58, C6, C7, C8, C9: value 100nF -> 100 nF
Connections:
- net Net-(U3-3V3) renamed ESP 3V3
- U1 pad 10: unconnected-(U1-VS_PLL-Pad10) -> GND
- U1 pad 11: unconnected-(U1-XOUT-Pad11) -> Net-(U1-XOUT)
- U1 pad 12: unconnected-(U1-XIN-Pad12) -> Net-(U1-XIN)
- U1 pad 13: unconnected-(U1-VD33-Pad13) -> HUB 3V3
- U1 pad 14: unconnected-(U1-DM4-Pad14) -> CON2 D-
- U1 pad 15: unconnected-(U1-DP4-Pad15) -> CON2 D+
- U1 pad 16: unconnected-(U1-VSS-Pad16) -> GND
- U1 pad 17: unconnected-(U1-DM3-Pad17) -> CON1 D-
- U1 pad 18: unconnected-(U1-DP3-Pad18) -> CON1 D+
- U1 pad 19: unconnected-(U1-VD33-Pad19) -> HUB 3V3
- U1 pad 20: unconnected-(U1-DM2-Pad20) -> ESP D-
- U1 pad 21: unconnected-(U1-DP2-Pad21) -> ESP D+
- U1 pad 22: unconnected-(U1-VSS-Pad22) -> GND
- U1 pad 23: unconnected-(U1-DM1-Pad23) -> STM D-
- U1 pad 24: unconnected-(U1-DP1-Pad24) -> STM D+
- U1 pad 25: unconnected-(U1-VS_A-Pad25) -> GND
- U1 pad 26: unconnected-(U1-VREG18-Pad26) -> HUB 1V8
- U1 pad 27: unconnected-(U1-VD3_IN-Pad27) -> HUB 3V3
- U1 pad 28: unconnected-(U1-REXT-Pad28) -> Net-(U1-REXT)
- U1 pad 29: unconnected-(U1-VD18-Pad29) -> HUB 1V8
- U1 pad 3: unconnected-(U1-VD18-Pad3) -> HUB 1V8
- U1 pad 30: unconnected-(U1-DMU-Pad30) -> HUB D-
- U1 pad 31: unconnected-(U1-DPU-Pad31) -> HUB D+
- U1 pad 32: unconnected-(U1-VD33-Pad32) -> HUB 3V3
- U1 pad 33: unconnected-(U1-VSS-Pad33) -> GND
- U1 pad 34: unconnected-(U1-XRSTJ-Pad34) -> Net-(U1-XRSTJ)
- U1 pad 35: unconnected-(U1-VBUSM-Pad35) -> +5V
- U1 pad 37: unconnected-(U1-DIS_REG-Pad37) -> Net-(U1-DIS_REG)
- U1 pad 38: unconnected-(U1-VD5_IN-Pad38) -> +5V
- U1 pad 39: unconnected-(U1-VD33_OUT-Pad39) -> HUB 3V3
- U1 pad 4: unconnected-(U1-PWRB[3]-Pad4) -> PWRB3
- U1 pad 40: unconnected-(U1-TEST-Pad40) -> GND
- U1 pad 41: unconnected-(U1-VD33-Pad41) -> HUB 3V3
- U1 pad 42: unconnected-(U1-DRV-Pad42) -> Net-(D60-K)
- U1 pad 43: unconnected-(U1-LED[1]-Pad43) -> Net-(U1-LED[1])
- U1 pad 44: unconnected-(U1-LED[2]-Pad44) -> Net-(U1-LED[2])
- U1 pad 45: unconnected-(U1-LED[3]-Pad45) -> Net-(U1-LED[3])
- U1 pad 46: unconnected-(U1-LED[4]-Pad46) -> Net-(U1-LED[4])
- U1 pad 5: unconnected-(U1-OVCB[3]-Pad5) -> OVCB3
- U1 pad 6: unconnected-(U1-VSS-Pad6) -> GND
- U1 pad 7: unconnected-(U1-OVCB[4]-Pad7) -> OVCB4
- U1 pad 8: unconnected-(U1-PWRB[4]-Pad8) -> PWRB4
- U1 pad 9: unconnected-(U1-VD_PLL-Pad9) -> HUB 1V8
- U3 pad 13: unconnected-(U3-GPIO19/U1RTS/ADC2_CH8/CLK_OUT2/USB_D--Pad13) -> ESP D-
- U3 pad 14: unconnected-(U3-GPIO20/U1CTS/ADC2_CH9/CLK_OUT1/USB_D+-Pad14) -> ESP D+
- U3 pad 27: unconnected-(U3-GPIO0/BOOT-Pad27) -> Net-(U3-GPIO0/BOOT)
- U3 pad 3: unconnected-(U3-EN-Pad3) -> ESP EN
- U3 pad 32: unconnected-(U3-MTCK/GPIO39/CLK_OUT3/SUBSPICS1-Pad32) -> Net-(J1-Pin_1)
- U3 pad 33: unconnected-(U3-MTDO/GPIO40/CLK_OUT2-Pad33) -> Net-(J1-Pin_2)
- U3 pad 34: unconnected-(U3-MTDI/GPIO41/CLK_OUT1-Pad34) -> Net-(J1-Pin_3)
- U3 pad 35: unconnected-(U3-MTMS/GPIO42-Pad35) -> Net-(J1-Pin_4)
- U3 pad 36: unconnected-(U3-U0RXD/GPIO44/CLK_OUT2-Pad36) -> Net-(J3-Pin_2)
- U3 pad 37: unconnected-(U3-U0TXD/GPIO43/CLK_OUT1-Pad37) -> Net-(J3-Pin_3)
- U3 pad 8: unconnected-(U3-GPIO15/U0RTS/ADC2_CH4/XTAL_32K_P-Pad8) -> Net-(U3-GPIO15/U0RTS/ADC2_CH4/XTAL_32K_P)
- U3 pad 9: unconnected-(U3-GPIO16/U0CTS/ADC2_CH5/XTAL_32K_N-Pad9) -> Net-(U3-GPIO16/U0CTS/ADC2_CH5/XTAL_32K_N)

Commit message: Initial wiring sorted out?
Parts:
- added U4: MX25R3235FM1xx1, Package_SO:SOP-8_3.9x4.9mm_P1.27mm, F.Cu at (267.0, 174.8)
Connections:
- U2 pad 10: Net-(U2-VSS-Pad10) -> GND
- U2 pad 100: unconnected-(U2-VDD-Pad100) -> STM 3V3
- U2 pad 11: unconnected-(U2-VDD-Pad11) -> STM 3V3
- U2 pad 12: unconnected-(U2-PH0-Pad12) -> Net-(U2-PH0)
- U2 pad 13: unconnected-(U2-PH1-Pad13) -> Net-(U2-PH1)
- U2 pad 14: unconnected-(U2-NRST-Pad14) -> STM Rst
- U2 pad 15: unconnected-(U2-PC0-Pad15) -> LCD_R5
- U2 pad 19: unconnected-(U2-VSSA-Pad19) -> GND
- U2 pad 20: unconnected-(U2-VREF+-Pad20) -> STM 3V3
- U2 pad 21: unconnected-(U2-VDDA-Pad21) -> STM 3V3
- U2 pad 23: unconnected-(U2-PA1-Pad23) -> LCD_R2
- U2 pad 24: unconnected-(U2-PA2-Pad24) -> LCD_R1
- U2 pad 25: unconnected-(U2-PA3-Pad25) -> LCD_B5
- U2 pad 26: Net-(U2-VSS-Pad10) -> GND
- U2 pad 27: unconnected-(U2-VDD-Pad27) -> STM 3V3
- U2 pad 28: unconnected-(U2-PA4-Pad28) -> LCD_VSYNC
- U2 pad 29: unconnected-(U2-PA5-Pad29) -> LCD_R4
- U2 pad 3: unconnected-(U2-PE4-Pad3) -> LCD_B0
- U2 pad 30: unconnected-(U2-PA6-Pad30) -> LCD_G2
- U2 pad 34: unconnected-(U2-PB0-Pad34) -> LCD_R3
- U2 pad 35: unconnected-(U2-PB1-Pad35) -> LCD_R6
- U2 pad 4: unconnected-(U2-PE5-Pad4) -> LCD_G0
- U2 pad 41: unconnected-(U2-PE11-Pad41) -> LCD_G3
- U2 pad 42: unconnected-(U2-PE12-Pad42) -> LCD_B4
- U2 pad 43: unconnected-(U2-PE13-Pad43) -> LCD_DE
- U2 pad 44: unconnected-(U2-PE14-Pad44) -> LCD_CLK
- U2 pad 45: unconnected-(U2-PE15-Pad45) -> LCD_R7
- U2 pad 46: unconnected-(U2-PB10-Pad46) -> LCD_G4
- U2 pad 47: unconnected-(U2-PB11-Pad47) -> LCD_G5
- U2 pad 48: unconnected-(U2-VCAP-Pad48) -> Net-(C81-Pad2)
- U2 pad 49: Net-(U2-VSS-Pad10) -> GND
- U2 pad 5: unconnected-(U2-PE6-Pad5) -> LCD_G1
- U2 pad 50: unconnected-(U2-VDD-Pad50) -> STM 3V3
- U2 pad 53: unconnected-(U2-PB14-Pad53) -> SD D0
- U2 pad 54: unconnected-(U2-PB15-Pad54) -> SD D1
- U2 pad 57: unconnected-(U2-PD10-Pad57) -> LCD_B3
- U2 pad 6: unconnected-(U2-VBAT-Pad6) -> STM 3V3
- U2 pad 63: unconnected-(U2-PC6-Pad63) -> LCD_HSYNC
- U2 pad 64: unconnected-(U2-PC7-Pad64) -> LCD_G6
- U2 pad 66: unconnected-(U2-PC9-Pad66) -> LCD_B2
- U2 pad 69: unconnected-(U2-PA10-Pad69) -> LCD_B1
- U2 pad 70: unconnected-(U2-PA11-Pad70) -> STM D-
- U2 pad 71: unconnected-(U2-PA12-Pad71) -> STM D+
- U2 pad 72: unconnected-(U2-PA13-Pad72) -> Net-(U2-PA13)
- U2 pad 73: unconnected-(U2-VCAP-Pad73) -> Net-(C80-Pad1)
- U2 pad 74: Net-(U2-VSS-Pad10) -> GND
- U2 pad 75: unconnected-(U2-VDD-Pad75) -> STM 3V3
- U2 pad 76: unconnected-(U2-PA14-Pad76) -> Net-(U2-PA14)
- U2 pad 8: unconnected-(U2-PC14-Pad8) -> Net-(U2-PC14)
- U2 pad 84: unconnected-(U2-PD3-Pad84) -> LCD_G7
- U2 pad 87: unconnected-(U2-PD6-Pad87) -> SD CK
- U2 pad 88: unconnected-(U2-PD7-Pad88) -> SD CMD
- U2 pad 89: unconnected-(U2-PB3-Pad89) -> SD D2
- U2 pad 9: unconnected-(U2-PC15-Pad9) -> Net-(U2-PC15)
- U2 pad 90: unconnected-(U2-PB4-Pad90) -> SD D3
- U2 pad 94: unconnected-(U2-BOOT0-Pad94) -> STM Boot
- U2 pad 95: unconnected-(U2-PB8-Pad95) -> LCD_B6
- U2 pad 96: unconnected-(U2-PB9-Pad96) -> LCD_B7
- U2 pad 99: Net-(U2-VSS-Pad10) -> GND

Commit message: Hub wired(?) + STM and ESP may boot already
Parts:
- added C59: 22u, Capacitor_SMD:C_0402_1005Metric_Pad0.74x0.62mm_HandSolder, F.Cu at (135.3, 113.6)
- added C60: 0.1u, Capacitor_SMD:C_0402_1005Metric_Pad0.74x0.62mm_HandSolder, F.Cu at (135.3, 116.9)
- added C61: C, Capacitor_SMD:C_0402_1005Metric_Pad0.74x0.62mm_HandSolder, F.Cu at (135.3, 120.3)
- added C62: C, Capacitor_SMD:C_0402_1005Metric_Pad0.74x0.62mm_HandSolder, F.Cu at (135.3, 123.6)
- added C63: 10u, Capacitor_SMD:C_0402_1005Metric_Pad0.74x0.62mm_HandSolder, F.Cu at (551.7, 274.4)
- added C64: 100n, Capacitor_SMD:C_0402_1005Metric_Pad0.74x0.62mm_HandSolder, B.Cu at (562.3, 276.5)
- added C65: 100n, Capacitor_SMD:C_0402_1005Metric_Pad0.74x0.62mm_HandSolder, F.Cu at (115.3, 120.3)
- added C66: 12p, Capacitor_SMD:C_0402_1005Metric_Pad0.74x0.62mm_HandSolder, F.Cu at (561.2, 284.5)
- added C67: 12p, Capacitor_SMD:C_0402_1005Metric_Pad0.74x0.62mm_HandSolder, F.Cu at (564.4, 282.0)
- added C68: 100n, Capacitor_SMD:C_0402_1005Metric_Pad0.74x0.62mm_HandSolder, B.Cu at (562.3, 279.5)
- added C69: 100n, Capacitor_SMD:C_0402_1005Metric_Pad0.74x0.62mm_HandSolder, B.Cu at (560.0, 272.7)
- added C70: 100n, Capacitor_SMD:C_0402_1005Metric_Pad0.74x0.62mm_HandSolder, B.Cu at (554.2, 276.0)
- added C71: 100n, Capacitor_SMD:C_0402_1005Metric_Pad0.74x0.62mm_HandSolder, B.Cu at (557.5, 272.7)
- added C72: 10u, Capacitor_SMD:C_0402_1005Metric_Pad0.74x0.62mm_HandSolder, F.Cu at (562.6, 269.9)
- added C73: 100n, Capacitor_SMD:C_0402_1005Metric_Pad0.74x0.62mm_HandSolder, B.Cu at (559.0, 272.7)
- added C74: 100n, Capacitor_SMD:C_0402_1005Metric_Pad0.74x0.62mm_HandSolder, B.Cu at (559.5, 280.9)
- added C75: 100n, Capacitor_SMD:C_0402_1005Metric_Pad0.74x0.62mm_HandSolder, B.Cu at (556.5, 280.9)
- added C76: 12p, Capacitor_SMD:C_0402_1005Metric_Pad0.74x0.62mm_HandSolder, B.Cu at (578.1, 275.1)
- added C77: 12p, Capacitor_SMD:C_0402_1005Metric_Pad0.74x0.62mm_HandSolder, B.Cu at (576.6, 275.1)
- added C78: C, Capacitor_SMD:C_0402_1005Metric_Pad0.74x0.62mm_HandSolder, F.Cu at (135.3, 133.7)
- added C79: 0.1u, Capacitor_SMD:C_0402_1005Metric_Pad0.74x0.62mm_HandSolder, F.Cu at (135.3, 137.0)
- added C80: 2.2u, Capacitor_SMD:C_0402_1005Metric_Pad0.74x0.62mm_HandSolder, F.Cu at (577.6, 278.6)
- added C81: 2.2u, Capacitor_SMD:C_0402_1005Metric_Pad0.74x0.62mm_HandSolder, F.Cu at (156.0, 116.9)
- added C82: 8p, Capacitor_SMD:C_0402_1005Metric_Pad0.74x0.62mm_HandSolder, B.Cu at (590.2, 296.0)
- added C83: 8p, Capacitor_SMD:C_0402_1005Metric_Pad0.74x0.62mm_HandSolder, B.Cu at (588.4, 297.6)
- added C84: 100n, Capacitor_SMD:C_0402_1005Metric_Pad0.74x0.62mm_HandSolder, F.Cu at (589.3, 286.4)
- added C85: 1.5p, Capacitor_SMD:C_0402_1005Metric_Pad0.74x0.62mm_HandSolder, B.Cu at (592.0, 295.3)
- added C86: 1.5p, Capacitor_SMD:C_0402_1005Metric_Pad0.74x0.62mm_HandSolder, B.Cu at (593.0, 294.3)
- added C87: 100n, Capacitor_SMD:C_0402_1005Metric_Pad0.74x0.62mm_HandSolder, F.Cu at (578.4, 277.9)
- added C88: 100n, Capacitor_SMD:C_0402_1005Metric_Pad0.74x0.62mm_HandSolder, F.Cu at (587.5, 290.5)
- added C89: 100n, Capacitor_SMD:C_0402_1005Metric_Pad0.74x0.62mm_HandSolder, F.Cu at (582.1, 295.8)
- added C90: 100n, Capacitor_SMD:C_0402_1005Metric_Pad0.74x0.62mm_HandSolder, F.Cu at (578.1, 296.9)
- added C91: 100n, Capacitor_SMD:C_0402_1005Metric_Pad0.74x0.62mm_HandSolder, F.Cu at (569.9, 288.8)
- added C92: 100n, Capacitor_SMD:C_0402_1005Metric_Pad0.74x0.62mm_HandSolder, F.Cu at (585.7, 292.3)
- added J1: ESP JTAG, Connector_PinHeader_2.54mm:PinHeader_1x04_P2.54mm_Vertical_SMD_Pin1Right, F.Cu at (576.0, 242.7)
- added J2: USB Connector, PCM_marbastlib-various:USB_C_Receptacle_HRO_TYPE-C-31-M-12, F.Cu at (558.4, 255.5)
- added J3: ESP UART, Connector_PinHeader_2.54mm:PinHeader_1x04_P2.54mm_Vertical_SMD_Pin1Right, F.Cu at (588.0, 242.7)
- added J5: Conn_01x40, Connector_FFC-FPC:TE_4-1734839-0_1x40-1MP_P0.5mm_Horizontal, F.Cu at (397.6, 340.4)
- added J7: STM Debug, Connector_PinHeader_2.54mm:PinHeader_1x04_P2.54mm_Vertical_SMD_Pin1Right, F.Cu at (579.7, 286.2)
- added R1: R, Resistor_SMD:R_0402_1005Metric_Pad0.72x0.64mm_HandSolder, F.Cu at (115.3, 130.3)
- added R10: R, Resistor_SMD:R_0402_1005Metric_Pad0.72x0.64mm_HandSolder, F.Cu at (557.0, 289.0)
- added R11: 5K1, Resistor_SMD:R_0402_1005Metric_Pad0.72x0.64mm_HandSolder, F.Cu at (560.1, 266.9)
- added R12: 5K1, Resistor_SMD:R_0402_1005Metric_Pad0.72x0.64mm_HandSolder, F.Cu at (556.5, 266.9)
- added R13: 10K, Resistor_SMD:R_0402_1005Metric_Pad0.72x0.64mm_HandSolder, F.Cu at (551.7, 273.3)
- added R14: NC, Resistor_SMD:R_0402_1005Metric_Pad0.72x0.64mm_HandSolder, F.Cu at (148.0, 129.1)
- added R15: 10K, Resistor_SMD:R_0402_1005Metric_Pad0.72x0.64mm_HandSolder, F.Cu at (162.6, 126.9)
- added R16: 22R, Resistor_SMD:R_0402_1005Metric_Pad0.72x0.64mm_HandSolder, F.Cu at (581.3, 281.4)
- added R17: 22R, Resistor_SMD:R_0402_1005Metric_Pad0.72x0.64mm_HandSolder, F.Cu at (578.5, 281.4)
- added R18: 10K, Resistor_SMD:R_0402_1005Metric_Pad0.72x0.64mm_HandSolder, F.Cu at (470.4, 202.1)
- added R2: R, Resistor_SMD:R_0402_1005Metric_Pad0.72x0.64mm_HandSolder, F.Cu at (115.3, 133.6)
- added R3: R, Resistor_SMD:R_0402_1005Metric_Pad0.72x0.64mm_HandSolder, F.Cu at (115.3, 136.9)
- added R4: R, Resistor_SMD:R_0402_1005Metric_Pad0.72x0.64mm_HandSolder, F.Cu at (115.3, 140.2)
- added R5: R, Resistor_SMD:R_0402_1005Metric_Pad0.72x0.64mm_HandSolder, F.Cu at (121.2, 130.3)
- added R6: 2K7, Resistor_SMD:R_0402_1005Metric_Pad0.72x0.64mm_HandSolder, F.Cu at (561.5, 269.9)
- added R7: 10K, Resistor_SMD:R_0402_1005Metric_Pad0.72x0.64mm_HandSolder, F.Cu at (555.5, 270.5)
- added R8: R, Resistor_SMD:R_0402_1005Metric_Pad0.72x0.64mm_HandSolder, F.Cu at (559.5, 289.0)
- added R9: R, Resistor_SMD:R_0402_1005Metric_Pad0.72x0.64mm_HandSolder, F.Cu at (148.0, 125.8)
- added SW1: ESP Boot, Button_Switch_SMD:SW_Push_1P1T_NO_CK_KMR2, F.Cu at (572.2, 266.2)
- added SW2: ESP Rst, Button_Switch_SMD:SW_Push_1P1T_NO_CK_KMR2, F.Cu at (577.2, 266.2)
- added SW3: STM Boot, Button_Switch_SMD:SW_Push_1P1T_NO_CK_KMR2, F.Cu at (459.5, 198.0)
- added SW4: STM Rst, Button_Switch_SMD:SW_Push_1P1T_NO_CK_KMR2, F.Cu at (469.5, 198.0)
- added Y1: 12 MHz, Crystal:Crystal_SMD_2016-4Pin_2.0x1.6mm, F.Cu at (562.8, 283.4)
- added Y2: 32.768 KHz, Crystal:Crystal_SMD_2012-2Pin_2.0x1.2mm, B.Cu at (577.3, 272.9)
- added Y3: 25 MHz, Crystal:Crystal_SMD_2016-4Pin_2.0x1.6mm, B.Cu at (588.2, 295.6)
- added Y4: 32.768 KHz, Crystal:Crystal_SMD_2012-2Pin_2.0x1.2mm, B.Cu at (590.8, 293.3)
- C1, C10, C11, C12, C13, C14, C15, C16, C17, C18, C19, C2, C20, C21, C22, C23, C24, C25, C26, C27, C28, C29, C3, C30, C31, C32, C33, C34, C35, C36, C37, C38, C39, C4, C40, C41, C42, C43, C44, C45, C46, C47, C48, C49, C5, C50, C51, C52, C53, C54, C55, C56, C57, C58, C6, C7, C8, C9: value 100 nF -> 100n; moved to B.Cu
- D1, D10, D11, D12, D13, D14, D15, D16, D17, D18, D19, D2, D20, D21, D22, D23, D24, D25, D26, D27, D28, D29, D3, D30, D31, D32, D33, D34, D35, D36, D37, D38, D39, D4, D40, D41, D42, D43, D44, D45, D46, D47, D48, D49, D5, D50, D51, D52, D53, D54, D55, D56, D57, D58, D6, D7, D8, D9, LED1, LED10, LED11, LED12, LED13, LED14, LED15, LED16, LED17, LED18, LED19, LED2, LED20, LED21, LED22, LED23, LED24, LED25, LED26, LED27, LED28, LED29, LED3, LED30, LED31, LED32, LED33, LED34, LED35, LED36, LED37, LED38, LED39, LED4, LED40, LED41, LED42, LED43, LED44, LED45, LED46, LED47, LED48, LED49, LED5, LED50, LED51, LED52, LED53, LED54, LED55, LED56, LED57, LED58, LED6, LED7, LED8, LED9, MX1, MX10, MX11, MX12, MX13, MX14, MX15, MX16, MX17, MX18, MX19, MX2, MX20, MX21, MX22, MX23, MX24, MX25, MX26, MX27, MX28, MX29, MX3, MX30, MX31, MX32, MX33, MX34, MX35, MX36, MX37, MX38, MX39, MX4, MX40, MX41, MX42, MX43, MX44, MX45, MX46, MX47, MX48, MX49, MX5, MX50, MX51, MX52, MX53, MX54, MX55, MX56, MX57, MX58, MX6, MX7, MX8, MX9: moved to B.Cu
- U1: moved to F.Cu
- U4: value MX25R3235FM1xx1 -> QSPI Flash
- moved MX48 363.2 mm to (231.3, 470.2), turned to 180 degrees
- moved MX58 363.2 mm to (231.3, 489.3), turned to 180 degrees
- moved LED12 363.2 mm to (231.3, 418.1), turned to 180 degrees
- moved LED24 363.2 mm to (231.3, 437.2), turned to 180 degrees
- moved LED36 363.2 mm to (231.3, 456.2), turned to 180 degrees
- moved LED48 363.2 mm to (231.3, 475.3), turned to 180 degrees
- moved LED58 363.2 mm to (231.3, 494.3), turned to 180 degrees
- moved MX12 363.2 mm to (231.3, 413.1), turned to 180 degrees
- moved MX24 363.2 mm to (231.3, 432.1), turned to 180 degrees
- moved MX36 363.2 mm to (231.3, 451.2), turned to 180 degrees
- moved C12 354.3 mm to (236.7, 417.2)
- moved C24 354.3 mm to (236.7, 436.3)
- moved C36 354.3 mm to (236.7, 455.3)
- moved C48 354.3 mm to (236.7, 474.4)
- moved C58 354.3 mm to (236.7, 493.4)
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Connections:
- U1 pad 20: ESP D- -> STM D-
- U1 pad 21: ESP D+ -> STM D+
- U1 pad 23: STM D- -> ESP D-
- U1 pad 24: STM D+ -> ESP D+
- U2 pad 100: STM 3V3 -> +3V3
- U2 pad 11: STM 3V3 -> +3V3
- U2 pad 21: STM 3V3 -> +3V3
- U2 pad 27: STM 3V3 -> +3V3
- U2 pad 50: STM 3V3 -> +3V3
- U2 pad 6: STM 3V3 -> +3V3
- U2 pad 75: STM 3V3 -> +3V3
- U3 pad 2: ESP 3V3 -> +3V3
- U5 pad 1: PWRB3 -> PWRB4
- U5 pad 2: OVCB3 -> OVCB4
- U5 pad 3: OVCB4 -> OVCB3
- U5 pad 4: PWRB4 -> PWRB3
- U5 pad 5: CON2 VBUS -> CON1 VBUS
- U5 pad 8: CON1 VBUS -> CON2 VBUS
Routing:
- net STM D+: track 0.00 -> 16.3 mm, vias 0 -> 1
- net STM D-: track 0.00 -> 16.0 mm, vias 0 -> 1
- net HUB 3V3: track 0.00 -> 15.4 mm, vias 0 -> 5
- net Net-(J3-Pin_2): track 0.00 -> 14.6 mm, vias 0 -> 1
- net Net-(J1-Pin_4): track 0.00 -> 14.1 mm, vias 0 -> 1
- net Net-(J1-Pin_2): track 0.00 -> 12.8 mm, vias 0 -> 1
- net HUB 1V8: track 0.00 -> 11.7 mm, vias 0 -> 3
- net Net-(J3-Pin_3): track 0.00 -> 10.7 mm, vias 0 -> 1
- net ESP D-: track 0.00 -> 10.7 mm, vias 0 -> 1
- net Net-(J1-Pin_3): track 0.00 -> 10.0 mm, vias 0 -> 1
- net ESP D+: track 0.00 -> 9.43 mm, vias 0 -> 1
- net Net-(J1-Pin_1): track 0.00 -> 8.98 mm, vias 0 -> 1
- net Net-(U2-PC14): track 0.00 -> 6.79 mm
- net PWRB3: track 0.00 -> 6.75 mm
- net Net-(U2-PH0): track 0.00 -> 6.51 mm
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- added copper zone on B.Cu, net +5V
- added copper zone on B.Cu, net GND
- removed copper zone on F.Cu, net +5V
- removed copper zone on F.Cu, net GND
Other:
- board size 274.7 x 100.5 mm -> 546.7 x 432.2 mm

Commit message: (WIP) Tracing v2
Parts:
- removed C62: C, Capacitor_SMD:C_0402_1005Metric_Pad0.74x0.62mm_HandSolder
- removed R10, R2, R3, R4, R5, R8: R, Resistor_SMD:R_0402_1005Metric_Pad0.72x0.64mm_HandSolder
- removed R14: NC, Resistor_SMD:R_0402_1005Metric_Pad0.72x0.64mm_HandSolder
- removed U4: QSPI Flash, Package_SO:SOP-8_3.9x4.9mm_P1.27mm
- removed U5: MIC2026-2BM, Package_DIP:DIP-8_W7.62mm
- added D59: HUB LED, LED_SMD:LED_0402_1005Metric_Pad0.77x0.64mm_HandSolder, F.Cu at (626.8, 320.0)
- added F1: 750 mA, Fuse:Fuse_0402_1005Metric_Pad0.77x0.64mm_HandSolder, F.Cu at (639.2, 308.4)
- added J4: SD Card, Connector_Card:microSD_HC_Hirose_DM3AT-SF-PEJM5, F.Cu at (392.0, 372.8)
- added J6: LS0XX, Connector_FFC-FPC:Molex_54548-1071_1x10-1MP_P0.5mm_Horizontal, F.Cu at (414.6, 362.6)
- added L1: L_Ferrite, Inductor_SMD:L_0402_1005Metric_Pad0.77x0.64mm_HandSolder, F.Cu at (634.0, 305.9)
- added L2: L_Ferrite, Inductor_SMD:L_0402_1005Metric_Pad0.77x0.64mm_HandSolder, F.Cu at (639.2, 305.9)
- added TP1: TestPoint, TestPoint:TestPoint_Pad_D2.0mm, B.Cu at (644.4, 313.4)
- added TP2: TestPoint, TestPoint:TestPoint_Pad_D2.0mm, B.Cu at (646.7, 315.5)
- added TP3: TestPoint, TestPoint:TestPoint_Pad_D2.0mm, B.Cu at (627.1, 323.3)
- added TP4: TestPoint, TestPoint:TestPoint_Pad_D2.0mm, B.Cu at (627.2, 318.8)
- C1, C10, C11, C12, C13, C14, C15, C16, C17, C18, C19, C2, C20, C21, C22, C23, C24, C25, C26, C27, C28, C29, C3, C30, C31, C32, C33, C34, C35, C36, C37, C38, C39, C4, C40, C41, C42, C43, C44, C45, C46, C47, C48, C49, C5, C50, C51, C52, C53, C54, C55, C56, C57, C58, C6, C7, C8, C9: footprint Capacitor_SMD:C_1206_3216Metric_Pad1.33x1.80mm_HandSolder -> Capacitor_SMD:C_0402_1005Metric_Pad0.74x0.62mm_HandSolder
- C61: value C -> 10u
- C64, C68, C69, C70, C71, C73, C74, C75: moved to F.Cu
- C80, C81: moved to B.Cu
- J5: value Conn_01x40 -> LTDC Screen
- Y1: footprint Crystal:Crystal_SMD_2016-4Pin_2.0x1.6mm -> Crystal:Crystal_SMD_3225-4Pin_3.2x2.5mm
- moved C65 557.6 mm to (640.3, 308.4), turned to -90 degrees
- moved R1 547.9 mm to (629.3, 320.0), turned to 180 degrees
- moved C81 544.0 mm to (661.1, 318.8), turned to 135 degrees
- moved C61 531.6 mm to (629.3, 316.7)
- moved MX48 476.0 mm to (548.5, 115.2)
- moved MX58 476.0 mm to (548.5, 134.3)
- moved MX12 476.0 mm to (548.5, 58.1)
- moved MX36 476.0 mm to (548.5, 96.2)
- moved LED12 476.0 mm to (548.5, 63.2)
- moved LED24 476.0 mm to (548.5, 82.2)
- moved LED36 476.0 mm to (548.5, 101.3)
- moved LED48 476.0 mm to (548.5, 120.3)
- moved LED58 476.0 mm to (548.5, 139.4)
- moved MX24 476.0 mm to (548.5, 77.1)
- moved C12 471.9 mm to (545.8, 60.6), turned to 0 degrees
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Connections:
- C61 pad 2: ESP D- -> +5V
- MX1 pad 1: COL_0 -> Net-(D1-A)
- MX1 pad 2: Net-(D1-A) -> COL_0
- MX10 pad 1: COL_9 -> Net-(D10-A)
- MX10 pad 2: Net-(D10-A) -> COL_9
- MX11 pad 1: COL_10 -> Net-(D11-A)
- MX11 pad 2: Net-(D11-A) -> COL_10
- MX12 pad 1: COL_11 -> Net-(D12-A)
- MX12 pad 2: Net-(D12-A) -> COL_11
- MX13 pad 1: COL_0 -> Net-(D13-A)
- MX13 pad 2: Net-(D13-A) -> COL_0
- MX14 pad 1: COL_1 -> Net-(D14-A)
- MX14 pad 2: Net-(D14-A) -> COL_1
- MX15 pad 1: COL_2 -> Net-(D15-A)
- MX15 pad 2: Net-(D15-A) -> COL_2
- MX16 pad 1: COL_3 -> Net-(D16-A)
- MX16 pad 2: Net-(D16-A) -> COL_3
- MX17 pad 1: COL_4 -> Net-(D17-A)
- MX17 pad 2: Net-(D17-A) -> COL_4
- MX18 pad 1: COL_5 -> Net-(D18-A)
- MX18 pad 2: Net-(D18-A) -> COL_5
- MX19 pad 1: COL_6 -> Net-(D19-A)
- MX19 pad 2: Net-(D19-A) -> COL_6
- MX2 pad 1: COL_1 -> Net-(D2-A)
- MX2 pad 2: Net-(D2-A) -> COL_1
- MX20 pad 1: COL_7 -> Net-(D20-A)
- MX20 pad 2: Net-(D20-A) -> COL_7
- MX21 pad 1: COL_8 -> Net-(D21-A)
- MX21 pad 2: Net-(D21-A) -> COL_8
- MX22 pad 1: COL_9 -> Net-(D22-A)
- MX22 pad 2: Net-(D22-A) -> COL_9
- MX23 pad 1: COL_10 -> Net-(D23-A)
- MX23 pad 2: Net-(D23-A) -> COL_10
- MX24 pad 1: COL_11 -> Net-(D24-A)
- MX24 pad 2: Net-(D24-A) -> COL_11
- MX25 pad 1: COL_0 -> Net-(D25-A)
- MX25 pad 2: Net-(D25-A) -> COL_0
- MX26 pad 1: COL_1 -> Net-(D26-A)
- MX26 pad 2: Net-(D26-A) -> COL_1
- MX27 pad 1: COL_2 -> Net-(D27-A)
- MX27 pad 2: Net-(D27-A) -> COL_2
- MX28 pad 1: COL_3 -> Net-(D28-A)
- MX28 pad 2: Net-(D28-A) -> COL_3
- MX29 pad 1: COL_4 -> Net-(D29-A)
- MX29 pad 2: Net-(D29-A) -> COL_4
- MX3 pad 1: COL_2 -> Net-(D3-A)
- MX3 pad 2: Net-(D3-A) -> COL_2
- MX30 pad 1: COL_5 -> Net-(D30-A)
- MX30 pad 2: Net-(D30-A) -> COL_5
- MX31 pad 1: COL_6 -> Net-(D31-A)
- MX31 pad 2: Net-(D31-A) -> COL_6
- MX32 pad 1: COL_7 -> Net-(D32-A)
- MX32 pad 2: Net-(D32-A) -> COL_7
- MX33 pad 1: COL_8 -> Net-(D33-A)
- MX33 pad 2: Net-(D33-A) -> COL_8
- MX34 pad 1: COL_9 -> Net-(D34-A)
- MX34 pad 2: Net-(D34-A) -> COL_9
- MX35 pad 1: COL_10 -> Net-(D35-A)
- MX35 pad 2: Net-(D35-A) -> COL_10
- MX36 pad 1: COL_11 -> Net-(D36-A)
- MX36 pad 2: Net-(D36-A) -> COL_11
- MX37 pad 1: COL_0 -> Net-(D37-A)
- MX37 pad 2: Net-(D37-A) -> COL_0
- MX38 pad 1: COL_1 -> Net-(D38-A)
- MX38 pad 2: Net-(D38-A) -> COL_1
- MX39 pad 1: COL_2 -> Net-(D39-A)
- MX39 pad 2: Net-(D39-A) -> COL_2
- MX4 pad 1: COL_3 -> Net-(D4-A)
- MX4 pad 2: Net-(D4-A) -> COL_3
- MX40 pad 1: COL_3 -> Net-(D40-A)
- MX40 pad 2: Net-(D40-A) -> COL_3
- MX41 pad 1: COL_4 -> Net-(D41-A)
- MX41 pad 2: Net-(D41-A) -> COL_4
- MX42 pad 1: COL_5 -> Net-(D42-A)
- MX42 pad 2: Net-(D42-A) -> COL_5
- MX43 pad 1: COL_6 -> Net-(D43-A)
- MX43 pad 2: Net-(D43-A) -> COL_6
- MX44 pad 1: COL_7 -> Net-(D44-A)
- MX44 pad 2: Net-(D44-A) -> COL_7
- MX45 pad 1: COL_8 -> Net-(D45-A)
- MX45 pad 2: Net-(D45-A) -> COL_8
- MX46 pad 1: COL_9 -> Net-(D46-A)
- MX46 pad 2: Net-(D46-A) -> COL_9
- MX47 pad 1: COL_10 -> Net-(D47-A)
- MX47 pad 2: Net-(D47-A) -> COL_10
- MX48 pad 1: COL_11 -> Net-(D48-A)
- MX48 pad 2: Net-(D48-A) -> COL_11
- MX49 pad 1: COL_0 -> Net-(D49-A)
- MX49 pad 2: Net-(D49-A) -> COL_0
- MX5 pad 1: COL_4 -> Net-(D5-A)
- MX5 pad 2: Net-(D5-A) -> COL_4
- MX50 pad 1: COL_1 -> Net-(D50-A)
- MX50 pad 2: Net-(D50-A) -> COL_1
- MX51 pad 1: COL_2 -> Net-(D51-A)
- MX51 pad 2: Net-(D51-A) -> COL_2
- MX52 pad 1: COL_3 -> Net-(D52-A)
- MX52 pad 2: Net-(D52-A) -> COL_3
- MX53 pad 1: COL_4 -> Net-(D53-A)
- MX53 pad 2: Net-(D53-A) -> COL_4
- MX54 pad 1: COL_6 -> Net-(D54-A)
- MX54 pad 2: Net-(D54-A) -> COL_6
- MX55 pad 1: COL_8 -> Net-(D55-A)
- MX55 pad 2: Net-(D55-A) -> COL_8
- MX56 pad 1: COL_9 -> Net-(D56-A)
- MX56 pad 2: Net-(D56-A) -> COL_9
- MX57 pad 1: COL_10 -> Net-(D57-A)
- MX57 pad 2: Net-(D57-A) -> COL_10
- MX58 pad 1: COL_11 -> Net-(D58-A)
- MX58 pad 2: Net-(D58-A) -> COL_11
- MX6 pad 1: COL_5 -> Net-(D6-A)
- MX6 pad 2: Net-(D6-A) -> COL_5
- MX7 pad 1: COL_6 -> Net-(D7-A)
- MX7 pad 2: Net-(D7-A) -> COL_6
- MX8 pad 1: COL_7 -> Net-(D8-A)
- MX8 pad 2: Net-(D8-A) -> COL_7
- MX9 pad 1: COL_8 -> Net-(D9-A)
- MX9 pad 2: Net-(D9-A) -> COL_8
- U1 pad 1: unconnected-(U1-OVCB[2]-Pad1) -> GND
- U1 pad 14: CON2 D- -> ESP D-
- U1 pad 15: CON2 D+ -> ESP D+
- U1 pad 17: CON1 D- -> unconnected-(U1-DM3-Pad17)
- U1 pad 18: CON1 D+ -> unconnected-(U1-DP3-Pad18)
- U1 pad 20: STM D- -> unconnected-(U1-DM2-Pad20)
- U1 pad 21: STM D+ -> unconnected-(U1-DP2-Pad21)
- U1 pad 23: ESP D- -> STM D-
- U1 pad 24: ESP D+ -> STM D+
- U1 pad 36: unconnected-(U1-BUS_B-Pad36) -> GND
- U1 pad 4: PWRB3 -> unconnected-(U1-PWRB[3]-Pad4)
- U1 pad 43: Net-(U1-LED[1]) -> GND
- U1 pad 44: Net-(U1-LED[2]) -> GND
- U1 pad 45: Net-(U1-LED[3]) -> unconnected-(U1-LED[3]-Pad45)
- U1 pad 46: Net-(U1-LED[4]) -> unconnected-(U1-LED[4]-Pad46)
- U1 pad 48: unconnected-(U1-OVCB[1]-Pad48) -> GND
- U1 pad 5: OVCB3 -> GND
- U1 pad 7: OVCB4 -> GND
- U1 pad 8: PWRB4 -> GND
Routing:
- net ROW_3: track 190.5 -> 0.00 mm
- net ROW_2: track 190.5 -> 0.00 mm
- net ROW_1: track 190.5 -> 0.00 mm
- net ROW_0: track 190.5 -> 0.00 mm
- net ROW_4: track 171.4 -> 0.00 mm
- net COL_6: track 80.1 -> 0.00 mm
- net COL_4: track 80.1 -> 0.00 mm
- net COL_9: track 76.2 -> 0.00 mm
- net COL_3: track 76.2 -> 0.00 mm
- net COL_8: track 76.2 -> 0.00 mm
- net COL_2: track 76.2 -> 0.00 mm
- net COL_11: track 76.2 -> 0.00 mm
- net COL_0: track 76.2 -> 0.00 mm
- net COL_10: track 76.2 -> 0.00 mm
- net COL_1: track 76.2 -> 0.00 mm
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- added copper zone on F.Cu, net GND
- removed copper zone on B.Cu, net +5V
Other:
- board size 546.7 x 432.2 mm -> 96.5 x 41.5 mm
