File: kicad/pcb/stm_peripherals.kicad_sch (KiCad schematic)
At the start: 2 parts, among them J4 Micro_SD_Card_Det1, U4 MX25R3235FM1xx1

Commit message: Initial wiring sorted out?
Parts:
- added J6: Conn_01x40, symbol Connector_Generic:Conn_01x40
- J4: value Micro_SD_Card_Det1 -> SD Card
- U4: value MX25R3235FM1xx1 -> QSPI Flash
Connections:
- net +3V3: now also J6.4 (Pin_4)
- net GND: now also J6.29 (Pin_29), J6.3 (Pin_3), J6.36 (Pin_36)
- new net +5V: J6.1 (Pin_1), J6.2 (Pin_2)
- new net LCD_B0: J6.21 (Pin_21)
- new net LCD_B1: J6.22 (Pin_22)
- new net LCD_B2: J6.23 (Pin_23)
- new net LCD_B3: J6.24 (Pin_24)
- new net LCD_B4: J6.25 (Pin_25)
- new net LCD_B5: J6.26 (Pin_26)
- new net LCD_B6: J6.27 (Pin_27)
- new net LCD_B7: J6.28 (Pin_28)
- new net LCD_CLK: J6.30 (Pin_30)
- new net LCD_DE: J6.34 (Pin_34)
- new net LCD_G0: J6.13 (Pin_13)
- new net LCD_G1: J6.14 (Pin_14)
- new net LCD_G2: J6.15 (Pin_15)
- new net LCD_G3: J6.16 (Pin_16)
- new net LCD_G4: J6.17 (Pin_17)
- new net LCD_G5: J6.18 (Pin_18)
- new net LCD_G6: J6.19 (Pin_19)
- new net LCD_G7: J6.20 (Pin_20)
- new net LCD_HSYNC: J6.32 (Pin_32)
- new net LCD_R1: J6.6 (Pin_6)
- new net LCD_R2: J6.7 (Pin_7)
- new net LCD_R3: J6.8 (Pin_8)
- new net LCD_R4: J6.9 (Pin_9)
- new net LCD_R5: J6.10 (Pin_10)
- new net LCD_R6: J6.11 (Pin_11)
- new net LCD_R7: J6.12 (Pin_12)
- new net LCD_VSYNC: J6.33 (Pin_33)
- no-connect marks 0 -> 1

Commit message: Hub wired(?) + STM and ESP may boot already
Parts:
- J6: footprint (none) -> Connector_FFC-FPC:TE_4-1734839-0_1x40-1MP_P0.5mm_Horizontal
Changed lines of the file:
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@@
       (effects (font (size 1.27 1.27)) (justify left))
     )
-    (property "Footprint" "" (at 257.81 92.71 0)
+    (property "Footprint" "Connector_FFC-FPC:TE_4-1734839-0_1x40-1MP_P0.5mm_Horizontal" (at 257.81 92.71 0)
       (effects (font (size 1.27 1.27)) hide)
     )

Commit message: (WIP) Tracing v2
Parts:
- removed U4: QSPI Flash, Package_SO:SOP-8_3.9x4.9mm_P1.27mm, symbol Memory_Flash:MX25R3235FM1xx1
- J4: footprint (none) -> Connector_Card:microSD_HC_Hirose_DM3AT-SF-PEJM5
- J6: value Conn_01x40 -> LTDC Screen
Other:
- moved on the sheet: J4, J6
